File: artificial-emotion-controller-v1/artificial-emotion-controller-v1.kicad_pcb (KiCad board)
At the start: 2 copper layers, 56.5 x 76.5 mm, 27 parts, among them J1 28BYJ-48 5-pin, J2 5V screw terminal, J8 I2C 3V3, U1 ESP32-S3 SuperMini, U2 ULN2003A

Commit message: Renumber controller v1 references and refresh the PCB.
Co-authored-by: Cursor <cursoragent@cursor.com>
Parts:
- SW1: renamed from BTN · IO7
- renumbered IO4 to J3, IO5 to J4, IO6 to J5, IO1 to J6, IO2 to J7, R5 to R1, R6 to R2, R7 to R3, R8 to R4, R9 to R5, R10 to R6, R12 to R7
Other:
- board text added: "BTN IO7"
- board text added: "ESP32"
- board text added: "IO1"
- board text added: "IO2"
- board text added: "IO4"
- board text added: "IO5"
- board text added: "IO6"
- board text added: "MOTOR"
- board text added: "R7"
Changed lines of the file:
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@@
 		(descr "Through hole straight pin header, 1x03, 2.54mm pitch, single row")
 		(tags "Through hole pin header THT 1x03 2.54mm single row")
-		(property "Reference" "IO6"
+		(property "Reference" "J5"
 			(at 0 7.5 90)
 			(layer "F.SilkS")
+			(hide yes)
 			(effects
 				(font
@@
 		(descr "Through hole straight pin header, 1x03, 2.54mm pitch, single row")
 		(tags "Through hole pin header THT 1x03 2.54mm single row")
-		(property "Reference" "IO4"
+		(property "Reference" "J3"
 			(at 0 7.5 90)
 			(layer "F.SilkS")
+			(hide yes)
 			(effects
 				(font
@@
 		(descr "Resistor, Axial_DIN0207 series, Axial, Horizontal, pin pitch=7.62mm, 0.25W = 1/4W, length*diameter=6.3*2.5mm^2, http://cdn-reichelt.de/documents/datenblatt/B400/1_4W%23YAG.pdf")
 		(tags "Resistor Axial_DIN0207 series Axial Horizontal pin pitch 7.62mm 0.25W = 1/4W length 6.3mm diameter 2.5mm")
-		(property "Reference" "R8"
-			(at 3.81 -2.37 0)
+		(property "Reference" "R4"
+			(at 3.81 -1 0)
 			(layer "F.SilkS")
 			(effects
@@
 		(descr "Resistor, Axial_DIN0207 series, Axial, Horizontal, pin pitch=7.62mm, 0.25W = 1/4W, length*diameter=6.3*2.5mm^2, http://cdn-reichelt.de/documents/datenblatt/B400/1_4W%23YAG.pdf")
 		(tags "Resistor Axial_DIN0207 series Axial Horizontal pin pitch 7.62mm 0.25W = 1/4W length 6.3mm diameter 2.5mm")
-		(property "Reference" "R12"
+		(property "Reference" "R7"
 			(at 3.81 -2.37 0)
 			(layer "F.SilkS")
@@
 		(descr "Resistor, Axial_DIN0207 series, Axial, Horizontal, pin pitch=7.62mm, 0.25W = 1/4W, length*diameter=6.3*2.5mm^2, http://cdn-reichelt.de/documents/datenblatt/B400/1_4W%23YAG.pdf")
 		(tags "Resistor Axial_DIN0207 series Axial Horizontal pin pitch 7.62mm 0.25W = 1/4W length 6.3mm diameter 2.5mm")
-		(property "Reference" "R7"
-			(at 3.81 -2.37 0)
+		(property "Reference" "R3"
+			(at 3.81 -1 0)
 			(layer "F.SilkS")
 			(effects
@@
 		(descr "Resistor, Axial_DIN0207 series, Axial, Horizontal, pin pitch=7.62mm, 0.25W = 1/4W, length*diameter=6.3*2.5mm^2, http://cdn-reichelt.de/documents/datenblatt/B400/1_4W%23YAG.pdf")
 		(tags "Resistor Axial_DIN0207 series Axial Horizontal pin pitch 7.62mm 0.25W = 1/4W length 6.3mm diameter 2.5mm")
-		(property "Reference" "R10"
+		(property "Reference" "R6"
 			(at 3.81 -2.37 0)
 			(layer "F.SilkS")
@@
 		(descr "Through hole straight pin header, 1x03, 2.54mm pitch, single row")
 		(tags "Through hole pin header THT 1x03 2.54mm single row")
-		(property "Reference" "IO2"
+		(property "Reference" "J7"
 			(at 0 7.54 90)
 			(layer "F.SilkS")
+			(hide yes)
 			(effects
 				(font
@@
 		(descr "Resistor, Axial_DIN0207 series, Axial, Horizontal, pin pitch=7.62mm, 0.25W = 1/4W, length*diameter=6.3*2.5mm^2, http://cdn-reichelt.de/documents/datenblatt/B400/1_4W%23YAG.pdf")
 		(tags "Resistor Axial_DIN0207 series Axial Horizontal pin pitch 7.62mm 0.25W = 1/4W length 6.3mm diameter 2.5mm")
-		(property "Reference" "R9"
-			(at 3.81 -2.37 0)
+		(property "Reference" "R5"
+			(at 3.81 -0.5 0)
 			(layer "F.SilkS")
 			(effects
@@
 		(descr "Through hole straight pin header, 1x03, 2.54mm pitch, single row")
 		(tags "Through hole pin header THT 1x03 2.54mm single row")
-		(property "Reference" "IO5"
+		(property "Reference" "J4"
 			(at 0 7.5 90)
 			(layer "F.SilkS")
+			(hide yes)
 			(effects
 				(font
@@
 		(descr "Through hole straight pin header, 1x03, 2.54mm pitch, single row")
 		(tags "Through hole pin header THT 1x03 2.54mm single row")
-		(property "Reference" "IO1"
+		(property "Reference" "J6"
 			(at 0 7.54 90)
 			(layer "F.SilkS")
+			(hide yes)
 			(effects
 				(font
@@
 			(at 0 -3.1425 0)
 			(layer "F.SilkS")
+			(hide yes)
 			(effects
 				(font
@@
 		(descr "Resistor, Axial_DIN0207 series, Axial, Horizontal, pin pitch=7.62mm, 0.25W = 1/4W, length*diameter=6.3*2.5mm^2, http://cdn-reichelt.de/documents/datenblatt/B400/1_4W%23YAG.pdf")
 		(tags "Resistor Axial_DIN0207 series Axial Horizontal pin pitch 7.62mm 0.25W = 1/4W length 6.3mm diameter 2.5mm")
-		(property "Reference" "R6"
+		(property "Reference" "R2"
 			(at 2.359781 0.12717 0)
 			(layer "F.SilkS")
@@
 		(descr "Generic 6mm SW tactile push button")
 		(tags "tact sw push 6mm")
-		(property "Reference" "BTN · IO7"
-			(at 3.25 -2.5 0)
+		(property "Reference" "SW1"
+			(at 3.25 2.25 0)
 			(layer "F.SilkS")
 			(effects
@@
 		(descr "Resistor, Axial_DIN0207 series, Axial, Horizontal, pin pitch=7.62mm, 0.25W = 1/4W, length*diameter=6.3*2.5mm^2, http://cdn-reichelt.de/documents/datenblatt/B400/1_4W%23YAG.pdf")
 		(tags "Resistor Axial_DIN0207 series Axial Horizontal pin pitch 7.62mm 0.25W = 1/4W length 6.3mm diameter 2.5mm")
-		(property "Reference" "R5"
+		(property "Reference" "R1"
 			(at 2.31 0 0)
 			(layer "F.SilkS")
@@
 			(at 0 -2.38 0)
 			(layer "F.SilkS")
+			(hide yes)
 			(effects
 				(font
@@
 		(tags "THT Terminal Block CUI TB007-508-02 pitch 5.08mm size 10.8x10.2mm drill 1.6mm pad 2.4mm")
 		(property "Reference" "J2"
-			(at 2.08 -7 0)
+			(at 2.84 -3.4 0)
 			(layer "F.SilkS")
 			(effects
@@
 	)
 	(gr_rect
-		(start 118.04 82)
+		(start 117.5 82)
 		(end 129.5 95.215306)
 		(stroke
@@
 	)
 	(gr_rect
-		(start 121.25 111)
+		(start 120.5 111)
 		(end 132.75 121.5)
 		(stroke
@@
 	)
 	(gr_rect
-		(start 121.296773 97.355933)
+		(start 120.832555 97.355933)
 		(end 132.756773 107.105933)
 		(stroke
@@
 		)
 	)
-	(gr_text "5V"
+	(gr_text "MOTOR\n"
+		(at 112 55.5 0)
+		(layer "F.SilkS")
+		(effects
+			(font
+				(size 0.8 0.8)
+				(thickness 0.1)
+			)
+		)
+	)
+	(gr_text "ESP32"
+		(at 117 55.5 0)
+		(layer "F.SilkS")
+		(effects
+			(font
+				(size 0.8 0.8)
+				(thickness 0.1)
+			)
+		)
+	)
+	(gr_text "GND\n"
 		(at 100 47.5 0)
 		(layer "F.SilkS")
@@
 		)
 	)
-	(gr_text "GND\n"
-		(at 107 47.5 0)
+	(gr_text "5V"
+		(at 106 47.5 0)
 		(layer "F.SilkS")
 		(effects
@@
 				(thickness 0.15)
 			)
+		)
+	)
+	(gr_text "BTN IO7"
+		(at 87 121 0)
+		(layer "F.SilkS")
+		(effects
+			(font
+				(size 1 1)
+				(thickness 0.1)
+			)
+			(justify left bottom)
+		)
+	)
+	(gr_text "IO6"
+		(at 119 86.5 90)
+		(layer "F.SilkS")
+		(effects
+			(font
+				(size 1 1)
+				(thickness 0.1)
+			)
+			(justify left bottom)
+		)
+	)
+	(gr_text "IO5"
+		(at 122.5 101 90)
+		(layer "F.SilkS")
+		(effects
+			(font
+				(size 1 1)
+				(thickness 0.1)
+			)
+			(justify left bottom)
+		)
+	)
+	(gr_text "IO4"
+		(at 122.5 105 90)
+		(layer "F.SilkS")
+		(effects
+			(font
+				(size 1 1)
+				(thickness 0.1)
+			)
+			(justify left bottom)
+		)
+	)
+	(gr_text "IO2"
+		(at 122.5 115 90)
+		(layer "F.SilkS")
+		(effects
+			(font
+				(size 1 1)
+				(thickness 0.1)
+			)
+			(justify left bottom)
+		)
+	)
+	(gr_text "IO1"
+		(at 122.5 119 90)
+		(layer "F.SilkS")
+		(effects
+			(font
+				(size 1 1)
+				(thickness 0.1)
+			)
+			(justify left bottom)
+		)
+	)
+	(gr_text "R7"
+		(at 103 64.5 0)
+		(layer "F.SilkS")
+		(effects
+			(font
+				(size 1 1)
+				(thickness 0.15)
+			)
