File: artificial-emotion-controller-v1/artificial-emotion-controller-v1.kicad_sch (KiCad schematic)
At the start: 31 parts, among them J1 28BYJ-48 5-pin, J2 5V screw terminal, J3 SENSOR A1 5V, J4 SENSOR A2 5V, J5 SENSOR A3 5V, J6 SENSOR B1 3V3, J7 SENSOR B2 3V3, J8 I2C 3V3, SW1 USER GPIO7 to GND, U1 ESP32-S3 SuperMini, U2 ULN2003A

Commit message: Revise controller v1 sensor banks, GPIO map, and fabrication files.
Bank A is now four 3.3V ports; the 5V divider is a single Bank B input.

Co-authored-by: Cursor <cursoragent@cursor.com>
Parts:
- removed R1, R3: 15K, Resistor_THT:R_Axial_DIN0207_L6.3mm_D2.5mm_P7.62mm_Horizontal, symbol PCM_SparkFun-Resistor:R
- removed R2, R4: 10K, Resistor_THT:R_Axial_DIN0207_L6.3mm_D2.5mm_P7.62mm_Horizontal, symbol PCM_SparkFun-Resistor:R
- J3: value SENSOR A1 5V -> SENSOR A3 3V3
- J4: value SENSOR A2 5V -> SENSOR A4 3V3
- J5: value SENSOR A3 5V -> SENSOR 5V
- J6: value SENSOR B1 3V3 -> SENSOR A1 3V3
- J7: value SENSOR B2 3V3 -> SENSOR A2 3V3
Connections:
- net ADC_A1 is gone; now on net SENSOR_A3: U1.6 (GPIO4)
- net ADC_A2 is gone; now on net SENSOR_A4: U1.7 (GPIO5)
- net 3V3: now also J3.2 (Pin_2), J4.2 (Pin_2)
- net 5V_MOTOR: no longer J3.2 (Pin_2), J4.2 (Pin_2)
- net SENSOR_A4: now reaches J4.3 (Pin_3)
- net SENSOR_A3: now reaches J3.3 (Pin_3)
- net ADC_A3 renamed SENSOR_B1_ADC
- net SENSOR_B1 renamed SENSOR_A1
- net SENSOR_B2 renamed SENSOR_A2
Other:
- moved on the sheet: J3, J4, J7, J8

Commit message: Renumber controller v1 references and refresh the PCB.
Co-authored-by: Cursor <cursoragent@cursor.com>
Parts:
- renumbered R5 to R1, R6 to R2, R7 to R3, R8 to R4, R9 to R5, R10 to R6, R12 to R7
Changed lines of the file:
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@@
 		(dnp no)
 		(fields_autoplaced yes)
-		(property "Reference" "R10"
+		(property "Reference" "R6"
 			(at 280.67 125.73 0)
 			(show_name no)
@@
 			(project "artificial-emotion-controller-v1"
 				(path "/50919683-80cf-4dee-9959-62511e3ef4ee"
-					(reference "R10")
+					(reference "R6")
 					(unit 1)
 				)
@@
 		(dnp no)
 		(fields_autoplaced yes)
-		(property "Reference" "R12"
+		(property "Reference" "R7"
 			(at 430.53 85.09 0)
 			(show_name no)
@@
 			(project "artificial-emotion-controller-v1"
 				(path "/50919683-80cf-4dee-9959-62511e3ef4ee"
-					(reference "R12")
+					(reference "R7")
 					(unit 1)
 				)
@@
 		(dnp no)
 		(fields_autoplaced yes)
-		(property "Reference" "R9"
+		(property "Reference" "R5"
 			(at 241.3 125.73 0)
 			(show_name no)
@@
 			(project "artificial-emotion-controller-v1"
 				(path "/50919683-80cf-4dee-9959-62511e3ef4ee"
-					(reference "R9")
+					(reference "R5")
 					(unit 1)
 				)
@@
 		(dnp no)
 		(fields_autoplaced yes)
-		(property "Reference" "R5"
+		(property "Reference" "R1"
 			(at 62.23 248.92 0)
 			(show_name no)
@@
 			(project "artificial-emotion-controller-v1"
 				(path "/50919683-80cf-4dee-9959-62511e3ef4ee"
-					(reference "R5")
+					(reference "R1")
 					(unit 1)
 				)
@@
 		(dnp no)
 		(fields_autoplaced yes)
-		(property "Reference" "R8"
+		(property "Reference" "R4"
 			(at 201.93 125.73 0)
 			(show_name no)
@@
 			(project "artificial-emotion-controller-v1"
 				(path "/50919683-80cf-4dee-9959-62511e3ef4ee"
-					(reference "R8")
+					(reference "R4")
 					(unit 1)
 				)
@@
 		(dnp no)
 		(fields_autoplaced yes)
-		(property "Reference" "R7"
+		(property "Reference" "R3"
 			(at 162.56 125.73 0)
 			(show_name no)
@@
 			(project "artificial-emotion-controller-v1"
 				(path "/50919683-80cf-4dee-9959-62511e3ef4ee"
-					(reference "R7")
+					(reference "R3")
 					(unit 1)
 				)
@@
 		(in_pos_files yes)
 		(dnp no)
-		(property "Reference" "R6"
+		(property "Reference" "R2"
 			(at 62.484 263.398 0)
 			(show_name no)
@@
 			(project "artificial-emotion-controller-v1"
 				(path "/50919683-80cf-4dee-9959-62511e3ef4ee"
-					(reference "R6")
-					(unit 1)
-				)
+					(reference "R2")
+					(unit 1)
+				)
